Commit message: 将激光雷达更新为360度扫描，修复了一些bug

File: catkin_ws/src/multi_robot_scenario/xacro/laser/hokuyo.xacro (robot description, xacro)
@@ -36,7 +36,7 @@
                 <!-- The URG-04LX-UG01  has  683 steps with 0.35139 Degree resolution -->
                 <resolution>1</resolution>
-                <max_angle>1.5708</max_angle> <!--2.0944 120 Degree -->
-                <min_angle>-1.5708</min_angle> <!-- -120 Degree -->
-                <samples>360</samples><!--<samples>683</samples>-->
+                <max_angle>3.14159</max_angle> <!-- 180 Degree (360° full circle) -->
+                <min_angle>-3.14159</min_angle> <!-- -180 Degree -->
+                <samples>720</samples><!--<samples>683</samples>-->
               </horizontal>
             </scan>

File: catkin_ws/src/multi_robot_scenario/xacro/p3dx/pioneer3dx.xacro (robot description, xacro)
@@ -8,5 +8,5 @@
   <!-- Laser -->
   <xacro:include filename="$(find multi_robot_scenario)/xacro/laser/hokuyo.xacro"/>
-  <xacro:laser name="front_laser" parent="chassis" xyz="0.125 0 0.25" rpy="0 0 0" meshes="package://gazebo_plugins/test/multi_robot_scenario/meshes/laser"/>
+  <xacro:laser name="front_laser" parent="chassis" xyz="0.125 0 0.45" rpy="0 0 0" meshes="package://gazebo_plugins/test/multi_robot_scenario/meshes/laser"/>
   <!-- GPU Laser
   <xacro:include filename="$(find multi_robot_scenario)/xacro/laser/hokuyo_gpu.xacro"/>
@@ -19,6 +19,6 @@
   <!-- Velodyne -->
   <xacro:include filename="$(find velodyne_description)/urdf/VLP-16.urdf.xacro"/>
-  <xacro:VLP-16 parent="base_link" name="velodyne" topic="/velodyne_points" hz="10" samples="360" gpu="false" min_angle="-1.57" max_angle="1.57" min_range="0.1">
-    <origin xyz="0.125 0 0.25" rpy="0 0 0" />
+  <xacro:VLP-16 parent="base_link" name="velodyne" topic="/velodyne_points" hz="10" samples="720" gpu="false" min_angle="-3.14159" max_angle="3.14159" min_range="0.3">
+    <origin xyz="0.125 0 0.5" rpy="0 0 0" />
   </xacro:VLP-16>
 </robot>
