Commit message: feat: 完善 c-space 训练与 ROS 导航支持

File: catkin_ws/src/multi_robot_scenario/xacro/p3dx/pioneer3dx.xacro (robot description, xacro)
@@ -8,5 +8,5 @@
   <!-- Laser -->
   <xacro:include filename="$(find multi_robot_scenario)/xacro/laser/hokuyo.xacro"/>
-  <xacro:laser name="front_laser" parent="chassis" xyz="0.125 0 0.45" rpy="0 0 0" meshes="package://gazebo_plugins/test/multi_robot_scenario/meshes/laser"/>
+  <xacro:laser name="front_laser" parent="chassis" xyz="0.125 0 0.26" rpy="0 0 0" meshes="package://gazebo_plugins/test/multi_robot_scenario/meshes/laser"/>
   <!-- GPU Laser
   <xacro:include filename="$(find multi_robot_scenario)/xacro/laser/hokuyo_gpu.xacro"/>
@@ -17,8 +17,3 @@
   <xacro:include filename="$(find multi_robot_scenario)/xacro/camera/cameraD.xacro"/>
   <xacro:camD name="cameraD" parent="chassis" xyz="0.025 0 0.32" rpy="0 0 0" />
-  <!-- Velodyne -->
-  <xacro:include filename="$(find velodyne_description)/urdf/VLP-16.urdf.xacro"/>
-  <xacro:VLP-16 parent="base_link" name="velodyne" topic="/velodyne_points" hz="10" samples="720" gpu="false" min_angle="-3.14159" max_angle="3.14159" min_range="0.3">
-    <origin xyz="0.125 0 0.5" rpy="0 0 0" />
-  </xacro:VLP-16>
 </robot>
