Commit message: feat(multi_robot_scenario): 机器人上方画出 cnav 的 c-space footprint
1.20 x 0.14 m，即 cnav_sparrow.yaml 的 footprint / settings.CSPACE_*，
挂在 base_link 上方 0.12 m（离地 0.27 m）。纯 visual，没有 collision、
没有 inertial，所以不影响物理。用来对比策略假设的车体尺寸和实际
0.13 x 0.12 m 的底盘。

File: catkin_ws/src/multi_robot_scenario/xacro/limo/limo_four_diff.xacro (robot description, xacro)
@@ -18,4 +18,10 @@
     <xacro:property name="wheel_length" value="0.045" />
     <xacro:property name="wheel_radius" value="0.045" />
+    <!-- The footprint the cnav policy plans with (settings.CSPACE_*), i.e. the
+         1.20 x 0.14 m rectangle in cnav_sparrow.yaml.  Drawn above the robot so
+         the assumed size can be compared against the real 0.13 x 0.12 m chassis. -->
+    <xacro:property name="cspace_footprint_x" value="1.20" />
+    <xacro:property name="cspace_footprint_y" value="0.14" />
+    <xacro:property name="cspace_footprint_z" value="0.12" />
   <link name="base_footprint"/>
   <joint name="base_joint" type="fixed">
@@ -39,4 +45,15 @@
           </geometry>
         </collision>
+        <!-- The cnav footprint.  Visual only, no collision, so it cannot change
+             how the robot drives. -->
+        <visual>
+            <origin xyz="0 0 ${cspace_footprint_z}" rpy="0 0 0" />
+            <geometry>
+                <box size="${cspace_footprint_x} ${cspace_footprint_y} 0.02"/>
+            </geometry>
+            <material name="cspace_footprint">
+                <color rgba="1.0 0.40 0.0 1.0"/>
+            </material>
+        </visual>
     </link>
     <!-- <link name="inertial_link">
